File: eagle/LAD_1_1.brd (EAGLE design)
At the start: 50 x 50 mm, 14 parts, among them X1 A1, X10 A, X2 A2, X3 A3, X4 A4, X5 A, X6 A1, X7 A2, X8 A3, X9 A4

Commit message: new boards (eagle files) and updated LAD_1_1 +DLS_1_0 +NOT_1_0 +PWR_1_0 +TFF_1_0 *LAD_1_1
Parts:
- X1, X6: value A1 -> A
- X10, X5: value A -> X
- X2, X7: value A2 -> B
- X3, X8: value A3 -> C
- X4, X9: value A4 -> D
Routing:
- net N$6: track 62.3 -> 61.1 mm
Other:
- board text added: "1"
- board text added: "4"
- board text added: "LAD v1.1"
- board text added: "Licensed under CERN OHL v.1.2"
- board text added: "www.mexdulon.com"
- board text removed: "E:/Bilder/Elektronik/Modulion/Mexdulon/mexdulon_50x50_pcb.bmp"
- board text removed: "Line Adapter v1.1"
