File: eagle/LAD_1_1.sch (EAGLE design)
At the start: 14 parts, among them X1 A1, X10 A, X2 A2, X3 A3, X4 A4, X5 A, X6 A1, X7 A2, X8 A3, X9 A4

Commit message: new boards (eagle files) and updated LAD_1_1 +DLS_1_0 +NOT_1_0 +PWR_1_0 +TFF_1_0 *LAD_1_1
Parts:
- X1, X6: value A1 -> A
- X10, X5: value A -> X
- X2, X7: value A2 -> B
- X3, X8: value A3 -> C
- X4, X9: value A4 -> D
Other:
- note added: "Copyright Oliver Krebs 2018"
- note removed: "Copyright Oliver Krebs 2017"
Changed lines of the file:
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@@
 <part name="GND1" library="supply1" deviceset="GND" device=""/>
 <part name="P+2" library="supply1" deviceset="VCC" device=""/>
-<part name="X1" library="01-my-con" deviceset="ML6D" device="" value="A1"/>
+<part name="X1" library="01-my-con" deviceset="ML6D" device="" value="A"/>
 <part name="H1" library="holes" deviceset="MOUNT-PAD-ROUND" device="3.2"/>
 <part name="H2" library="holes" deviceset="MOUNT-PAD-ROUND" device="3.2"/>
@@
 <part name="GND2" library="supply1" deviceset="GND" device=""/>
 <part name="P+1" library="supply1" deviceset="VCC" device=""/>
-<part name="X2" library="01-my-con" deviceset="ML6D" device="" value="A2"/>
+<part name="X2" library="01-my-con" deviceset="ML6D" device="" value="B"/>
 <part name="GND3" library="supply1" deviceset="GND" device=""/>
 <part name="P+3" library="supply1" deviceset="VCC" device=""/>
-<part name="X3" library="01-my-con" deviceset="ML6D" device="" value="A3"/>
+<part name="X3" library="01-my-con" deviceset="ML6D" device="" value="C"/>
 <part name="GND4" library="supply1" deviceset="GND" device=""/>
 <part name="P+4" library="supply1" deviceset="VCC" device=""/>
-<part name="X4" library="01-my-con" deviceset="ML6D" device="" value="A4"/>
+<part name="X4" library="01-my-con" deviceset="ML6D" device="" value="D"/>
 <part name="GND6" library="supply1" deviceset="GND" device=""/>
 <part name="P+5" library="supply1" deviceset="VCC" device=""/>
-<part name="X5" library="01-my-con" deviceset="ML6D" device="" value="A"/>
+<part name="X5" library="01-my-con" deviceset="ML6D" device="" value="X"/>
 <part name="GND7" library="supply1" deviceset="GND" device=""/>
 <part name="P+6" library="supply1" deviceset="VCC" device=""/>
-<part name="X6" library="01-my-con" deviceset="ML6D" device="" value="A1"/>
+<part name="X6" library="01-my-con" deviceset="ML6D" device="" value="A"/>
 <part name="GND8" library="supply1" deviceset="GND" device=""/>
 <part name="P+7" library="supply1" deviceset="VCC" device=""/>
-<part name="X7" library="01-my-con" deviceset="ML6D" device="" value="A2"/>
+<part name="X7" library="01-my-con" deviceset="ML6D" device="" value="B"/>
 <part name="GND9" library="supply1" deviceset="GND" device=""/>
 <part name="P+8" library="supply1" deviceset="VCC" device=""/>
-<part name="X8" library="01-my-con" deviceset="ML6D" device="" value="A3"/>
+<part name="X8" library="01-my-con" deviceset="ML6D" device="" value="C"/>
 <part name="GND10" library="supply1" deviceset="GND" device=""/>
 <part name="P+9" library="supply1" deviceset="VCC" device=""/>
-<part name="X9" library="01-my-con" deviceset="ML6D" device="" value="A4"/>
-<part name="X10" library="01-my-con" deviceset="ML6D" device="" value="A"/>
+<part name="X9" library="01-my-con" deviceset="ML6D" device="" value="D"/>
+<part name="X10" library="01-my-con" deviceset="ML6D" device="" value="X"/>
 <part name="P+10" library="supply1" deviceset="VCC" device=""/>
 <part name="GND11" library="supply1" deviceset="GND" device=""/>
@@
 <sheet>
 <plain>
-<text x="104.14" y="7.62" size="1.27" layer="97" distance="60">This documentation describes Open Hardware and is licensed
+<text x="91.44" y="5.08" size="1.778" layer="97" distance="60">This documentation describes Open Hardware and is licensed
 under the CERN OHL v. 1.2. You may redistribute and modify this
 documentation under the terms of the CERN OHL v.1.2.
@@
 QUALITY AND FITNESS FOR A PARTICULAR PURPOSE.
 Please see the CERN OHL v.1.2 for applicable conditions</text>
-<text x="166.37" y="25.4" size="2.1844" layer="94" distance="60">Copyright Oliver Krebs 2017</text>
+<text x="166.37" y="25.4" size="2.1844" layer="94" distance="60">Copyright Oliver Krebs 2018</text>
 </plain>
 <instances>
