File: eagle/RGB_1_1b.brd (EAGLE design)
At the start: 50 x 50 mm, 16 parts, among them X1 RGB, X2 Buzzer

Commit message: Missing doc files added, schematics.pdf created +doc/pdf/schematics.pdf: all schematics in one file
Parts:
- R2: value 4k7 -> 680
- R3: value 10k -> 4k7
- R4: value 2k2 -> 470
Changed lines of the file:
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@@
 <?xml version="1.0" encoding="utf-8"?>
 <!DOCTYPE eagle SYSTEM "eagle.dtd">
-<eagle version="7.6.0">
+<eagle version="8.3.2">
 <drawing>
 <settings>
 <setting alwaysvectorfont="no"/>
+<setting keepoldvectorfont="yes"/>
 <setting verticaltext="up"/>
 </settings>
@@
 </element>
 <element name="SG1" library="buzzer" package="F/CM12P" value="F/CM12P" x="33.02" y="13.97" smashed="yes" rot="R180">
+<attribute name="MF" value="" x="33.02" y="13.97" size="1.778" layer="27" rot="R180" display="off"/>
+<attribute name="MPN" value="" x="33.02" y="13.97" size="1.778" layer="27" rot="R180" display="off"/>
+<attribute name="NAME" x="32.1" y="8.62" size="1.27" layer="25" font="vector" ratio="10"/>
+<attribute name="OC_FARNELL" value="unknown" x="33.02" y="13.97" size="1.778" layer="27" rot="R180" display="off"/>
 <attribute name="OC_NEWARK" value="unknown" x="33.02" y="13.97" size="1.778" layer="27" rot="R180" display="off"/>
-<attribute name="MPN" value="" x="33.02" y="13.97" size="1.778" layer="27" rot="R180" display="off"/>
-<attribute name="MF" value="" x="33.02" y="13.97" size="1.778" layer="27" rot="R180" display="off"/>
-<attribute name="OC_FARNELL" value="unknown" x="33.02" y="13.97" size="1.778" layer="27" rot="R180" display="off"/>
-<attribute name="NAME" x="32.1" y="8.62" size="1.27" layer="25" font="vector" ratio="10"/>
 <attribute name="VALUE" x="37.465" y="17.78" size="1.27" layer="27" font="vector" ratio="10" rot="R180"/>
 </element>
@@
 <attribute name="VALUE" x="30.7594" y="29.845" size="1.016" layer="27" font="vector" ratio="10"/>
 </element>
-<element name="R2" library="01-my_rcl" package="0207/10" value="4k7" x="33.02" y="33.02" smashed="yes">
+<element name="R2" library="01-my_rcl" package="0207/10" value="680" x="33.02" y="33.02" smashed="yes">
 <attribute name="NAME" x="36.068" y="33.401" size="1.016" layer="25" font="vector" ratio="10" rot="R180"/>
 <attribute name="VALUE" x="30.7594" y="32.385" size="1.016" layer="27" font="vector" ratio="10"/>
 </element>
-<element name="R3" library="01-my_rcl" package="0207/10" value="10k" x="33.02" y="35.56" smashed="yes">
+<element name="R3" library="01-my_rcl" package="0207/10" value="4k7" x="33.02" y="35.56" smashed="yes">
 <attribute name="NAME" x="36.068" y="35.941" size="1.016" layer="25" font="vector" ratio="10" rot="R180"/>
 <attribute name="VALUE" x="30.7594" y="34.925" size="1.016" layer="27" font="vector" ratio="10"/>
 </element>
-<element name="R4" library="01-my_rcl" package="0207/10" value="2k2" x="33.02" y="38.1" smashed="yes">
+<element name="R4" library="01-my_rcl" package="0207/10" value="470" x="33.02" y="38.1" smashed="yes">
 <attribute name="NAME" x="36.068" y="38.481" size="1.016" layer="25" font="vector" ratio="10" rot="R180"/>
 <attribute name="VALUE" x="30.7594" y="37.465" size="1.016" layer="27" font="vector" ratio="10"/>
