File: eagle/LED_1_1.sch (EAGLE design)
At the start: 17 parts, among them X1 In B, X2 Out B, X3 In A, X4 Out A

Commit message: Add new tetra-Board and arduino files
Add AMP_1_0, AVC_1_0, D18_1_1, IOP_1_2, MIC_1_0, PIN_1_1, POT_1_0, PWA_1_0, PWR_1_0, RGF 2.0, SOC_2_0, VLT_1_0
Add mex_nano_shield_keyboard, mex_nano_shied_numbers

New arduino projects
Other:
- moved on the sheet: H1, H2, H3, H4, P1, P2, P3, P4, P5, P6, P7, P8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
